Commit message: some work

File: src/kinova-ros-kinetic/kinova_description/urdf/kinova_common.xacro (robot description, xacro)
@@ -113,5 +113,5 @@
             <axis xyz="0 0 1"/>
             <origin xyz="0.044 -0.003 0" rpy="0 0 0"/>
-            <limit lower="0" upper="2" effort="1" velocity="1"/>
+            <limit lower="0" upper="2.5" effort="1" velocity="1"/>
         </joint>
     </xacro:macro>
